File: esp-switch.sch (KiCad schematic (older format))
At the start: 21 parts, among them J1 Screw_Terminal_01x02, J2 Conn_01x04, J3 Screw_Terminal_01x02, J4 Conn_01x04, U1 ATTINY441-SSU, U2 ESP-01v090, U3 MOC3043M, U4 MOC3043M, U5 HLK-PM03

Commit message: V4 smaller PCB
Parts:
- removed J4: Conn_01x04, Pin_Headers:Pin_Header_Straight_1x04_Pitch2.54mm, symbol Conn_01x04
- R4: renamed from R5; footprint Resistors_THT:R_Axial_DIN0411_L9.9mm_D3.6mm_P5.08mm_Vertical -> Resistors_THT:R_Axial_DIN0207_L6.3mm_D2.5mm_P5.08mm_Vertical
- R5: renamed from R6; footprint Resistors_THT:R_Axial_DIN0411_L9.9mm_D3.6mm_P7.62mm_Vertical -> Resistors_THT:R_Axial_DIN0207_L6.3mm_D2.5mm_P5.08mm_Vertical
- R6: renamed from R7; footprint Resistors_THT:R_Axial_DIN0411_L9.9mm_D3.6mm_P5.08mm_Vertical -> Resistors_THT:R_Axial_DIN0207_L6.3mm_D2.5mm_P5.08mm_Vertical
- R7: renamed from R8; footprint Resistors_THT:R_Axial_DIN0411_L9.9mm_D3.6mm_P7.62mm_Vertical -> Resistors_THT:R_Axial_DIN0207_L6.3mm_D2.5mm_P5.08mm_Vertical
- renumbered D3 to D1, D4 to D2, J3 to J1, J1 to J2, J2 to J3, R9 to R1, R3 to R2, R4 to R3
Changed lines of the file:
@@
 $EndComp
 $Comp
-L R R3
+L R R2
 U 1 1 5A12ED7C
 P 8300 3450
-F 0 "R3" V 8380 3450 50  0000 C CNN
+F 0 "R2" V 8380 3450 50  0000 C CNN
 F 1 "150R" V 8300 3450 50  0000 C CNN
 F 2 "Resistors_THT:R_Axial_DIN0204_L3.6mm_D1.6mm_P2.54mm_Vertical" V 8230 3450 50  0001 C CNN
@@
 $EndComp
 $Comp
-L GND #PWR04
-U 1 1 5A12EDB6
-P 8100 3850
-F 0 "#PWR04" H 8100 3600 50  0001 C CNN
-F 1 "GND" H 8100 3700 50  0000 C CNN
-F 2 "" H 8100 3850 50  0001 C CNN
-F 3 "" H 8100 3850 50  0001 C CNN
-	1    8100 3850
-	1    0    0    -1
-$EndComp
-$Comp
-L TRIAC_TTG D3
+L TRIAC_TTG D1
 U 1 1 5A12F072
 P 9500 3000
-F 0 "D3" H 9625 3025 50  0000 L CNN
+F 0 "D1" H 9625 3025 50  0000 L CNN
 F 1 "BTA08-600BW" H 9625 2950 50  0000 L CNN
 F 2 "TO_SOT_Packages_THT:TO-220_Vertical" V 9575 3025 50  0001 C CNN
@@
 $EndComp
 $Comp
-L R R5
+L R R4
 U 1 1 5A12F124
 P 9250 2550
-F 0 "R5" V 9330 2550 50  0000 C CNN
+F 0 "R4" V 9330 2550 50  0000 C CNN
 F 1 "390R" V 9250 2550 50  0000 C CNN
-F 2 "Resistors_THT:R_Axial_DIN0411_L9.9mm_D3.6mm_P5.08mm_Vertical" V 9180 2550 50  0001 C CNN
+F 2 "Resistors_THT:R_Axial_DIN0207_L6.3mm_D2.5mm_P5.08mm_Vertical" V 9180 2550 50  0001 C CNN
 F 3 "" H 9250 2550 50  0001 C CNN
 	1    9250 2550
@@
 $EndComp
 $Comp
-L R R6
+L R R5
 U 1 1 5A12F2D1
 P 9250 3400
-F 0 "R6" V 9330 3400 50  0000 C CNN
+F 0 "R5" V 9330 3400 50  0000 C CNN
 F 1 "470R" V 9250 3400 50  0000 C CNN
-F 2 "Resistors_THT:R_Axial_DIN0411_L9.9mm_D3.6mm_P7.62mm_Vertical" V 9180 3400 50  0001 C CNN
+F 2 "Resistors_THT:R_Axial_DIN0207_L6.3mm_D2.5mm_P5.08mm_Vertical" V 9180 3400 50  0001 C CNN
 F 3 "" H 9250 3400 50  0001 C CNN
 	1    9250 3400
@@
 $EndComp
 $Comp
-L R R4
+L R R3
 U 1 1 5A132A9E
 P 8300 5300
-F 0 "R4" V 8380 5300 50  0000 C CNN
+F 0 "R3" V 8380 5300 50  0000 C CNN
 F 1 "150R" V 8300 5300 50  0000 C CNN
 F 2 "Resistors_THT:R_Axial_DIN0204_L3.6mm_D1.6mm_P2.54mm_Vertical" V 8230 5300 50  0001 C CNN
@@
 $EndComp
 $Comp
-L GND #PWR05
+L GND #PWR04
 U 1 1 5A132AA4
 P 8300 5600
-F 0 "#PWR05" H 8300 5350 50  0001 C CNN
+F 0 "#PWR04" H 8300 5350 50  0001 C CNN
 F 1 "GND" H 8300 5450 50  0000 C CNN
 F 2 "" H 8300 5600 50  0001 C CNN
@@
 $EndComp
 $Comp
-L TRIAC_TTG D4
+L TRIAC_TTG D2
 U 1 1 5A132AB3
 P 9500 4850
-F 0 "D4" H 9625 4875 50  0000 L CNN
+F 0 "D2" H 9625 4875 50  0000 L CNN
 F 1 "BTA08-600BW" H 9625 4800 50  0000 L CNN
 F 2 "TO_SOT_Packages_THT:TO-220_Vertical" V 9575 4875 50  0001 C CNN
@@
 $EndComp
 $Comp
-L R R7
+L R R6
 U 1 1 5A132AB9
 P 9250 4400
-F 0 "R7" V 9330 4400 50  0000 C CNN
+F 0 "R6" V 9330 4400 50  0000 C CNN
 F 1 "390R" V 9250 4400 50  0000 C CNN
-F 2 "Resistors_THT:R_Axial_DIN0411_L9.9mm_D3.6mm_P5.08mm_Vertical" V 9180 4400 50  0001 C CNN
+F 2 "Resistors_THT:R_Axial_DIN0207_L6.3mm_D2.5mm_P5.08mm_Vertical" V 9180 4400 50  0001 C CNN
 F 3 "" H 9250 4400 50  0001 C CNN
 	1    9250 4400
@@
 $EndComp
 $Comp
-L R R8
+L R R7
 U 1 1 5A132AC2
 P 9250 5250
-F 0 "R8" V 9330 5250 50  0000 C CNN
+F 0 "R7" V 9330 5250 50  0000 C CNN
 F 1 "470R" V 9250 5250 50  0000 C CNN
-F 2 "Resistors_THT:R_Axial_DIN0411_L9.9mm_D3.6mm_P7.62mm_Vertical" V 9180 5250 50  0001 C CNN
+F 2 "Resistors_THT:R_Axial_DIN0207_L6.3mm_D2.5mm_P5.08mm_Vertical" V 9180 5250 50  0001 C CNN
 F 3 "" H 9250 5250 50  0001 C CNN
 	1    9250 5250
 	0    1    1    0
-$EndComp
-$Comp
-L Conn_01x04 J4
-U 1 1 5A557EC8
-P 6850 3400
-F 0 "J4" H 6850 3600 50  0000 C CNN
-F 1 "Conn_01x04" H 6850 3100 50  0000 C CNN
-F 2 "Pin_Headers:Pin_Header_Straight_1x04_Pitch2.54mm" H 6850 3400 50  0001 C CNN
-F 3 "" H 6850 3400 50  0001 C CNN
-	1    6850 3400
-	-1   0    0    -1
 $EndComp
 $Comp
@@
 $EndComp
 $Comp
-L GND #PWR06
+L GND #PWR05
 U 1 1 5A55918B
 P 9050 1700
-F 0 "#PWR06" H 9050 1450 50  0001 C CNN
+F 0 "#PWR05" H 9050 1450 50  0001 C CNN
 F 1 "GND" H 9050 1550 50  0000 C CNN
 F 2 "" H 9050 1700 50  0001 C CNN
@@
 $EndComp
 $Comp
-L GND #PWR07
+L GND #PWR06
 U 1 1 5A669AF1
 P 8750 1700
-F 0 "#PWR07" H 8750 1450 50  0001 C CNN
+F 0 "#PWR06" H 8750 1450 50  0001 C CNN
 F 1 "GND" H 8750 1550 50  0000 C CNN
 F 2 "" H 8750 1700 50  0001 C CNN
@@
 $EndComp
 $Comp
-L +3.3V #PWR08
+L +3.3V #PWR07
 U 1 1 5A6DF18D
 P 8750 1350
-F 0 "#PWR08" H 8750 1200 50  0001 C CNN
+F 0 "#PWR07" H 8750 1200 50  0001 C CNN
 F 1 "+3.3V" H 8750 1490 50  0000 C CNN
 F 2 "" H 8750 1350 50  0001 C CNN
@@
 $EndComp
 $Comp
-L +3.3V #PWR09
+L +3.3V #PWR08
 U 1 1 5A6DF2D7
 P 9050 1450
-F 0 "#PWR09" H 9050 1300 50  0001 C CNN
+F 0 "#PWR08" H 9050 1300 50  0001 C CNN
 F 1 "+3.3V" H 9050 1590 50  0000 C CNN
 F 2 "" H 9050 1450 50  0001 C CNN
@@
 $EndComp
 $Comp
-L +3.3V #PWR010
+L +3.3V #PWR09
 U 1 1 5A6DF347
 P 7100 900
-F 0 "#PWR010" H 7100 750 50  0001 C CNN
+F 0 "#PWR09" H 7100 750 50  0001 C CNN
 F 1 "+3.3V" H 7100 1040 50  0000 C CNN
 F 2 "" H 7100 900 50  0001 C CNN
@@
 $EndComp
 $Comp
-L +3.3V #PWR011
-U 1 1 5A6DFFEC
-P 7400 3350
-F 0 "#PWR011" H 7400 3200 50  0001 C CNN
-F 1 "+3.3V" H 7400 3490 50  0000 C CNN
-F 2 "" H 7400 3350 50  0001 C CNN
-F 3 "" H 7400 3350 50  0001 C CNN
-	1    7400 3350
-	1    0    0    -1
-$EndComp
-$Comp
-L +3.3V #PWR012
+L +3.3V #PWR010
 U 1 1 5A6E0C46
 P 4050 2500
-F 0 "#PWR012" H 4050 2350 50  0001 C CNN
+F 0 "#PWR010" H 4050 2350 50  0001 C CNN
 F 1 "+3.3V" H 4050 2640 50  0000 C CNN
 F 2 "" H 4050 2500 50  0001 C CNN
@@
 $EndComp
 $Comp
-L +3.3V #PWR013
+L +3.3V #PWR011
 U 1 1 5A6E1A62
 P 1200 750
-F 0 "#PWR013" H 1200 600 50  0001 C CNN
+F 0 "#PWR011" H 1200 600 50  0001 C CNN
 F 1 "+3.3V" H 1200 890 50  0000 C CNN
 F 2 "" H 1200 750 50  0001 C CNN
@@
 $EndComp
 $Comp
-L Conn_01x04 J2
+L Conn_01x04 J3
 U 1 1 5A635AA5
 P 4750 750
-F 0 "J2" H 4750 950 50  0000 C CNN
+F 0 "J3" H 4750 950 50  0000 C CNN
 F 1 "Conn_01x04" H 4750 450 50  0000 C CNN
 F 2 "Pin_Headers:Pin_Header_Straight_1x04_Pitch2.54mm" H 4750 750 50  0001 C CNN
@@
 $EndComp
 $Comp
-L +3.3V #PWR014
+L +3.3V #PWR012
 U 1 1 5AEF4831
 P 6300 700
-F 0 "#PWR014" H 6300 550 50  0001 C CNN
+F 0 "#PWR012" H 6300 550 50  0001 C CNN
 F 1 "+3.3V" H 6300 840 50  0000 C CNN
 F 2 "" H 6300 700 50  0001 C CNN
@@
 $EndComp
 $Comp
-L R R9
+L R R1
 U 1 1 5AEF60B4
 P 6300 850
-F 0 "R9" V 6380 850 50  0000 C CNN
+F 0 "R1" V 6380 850 50  0000 C CNN
 F 1 "10K" V 6300 850 50  0000 C CNN
 F 2 "Resistors_THT:R_Axial_DIN0204_L3.6mm_D1.6mm_P2.54mm_Vertical" V 6230 850 50  0001 C CNN
@@
 	4150 3000 4050 3000
 Wire Wire Line
-	7350 3750 8300 3750
-Wire Wire Line
 	8300 3750 8300 3600
-Wire Wire Line
-	8100 3750 8100 3850
-Connection ~ 8100 3750
 Wire Wire Line
 	8300 3300 8300 3100
@@
 	9650 4400 9400 4400
 Wire Wire Line
-	7150 3300 7050 3300
-Wire Wire Line
-	7150 2000 7150 3300
-Wire Wire Line
-	7050 3400 7150 3400
-Wire Wire Line
-	7150 3400 7150 4400
-Wire Wire Line
-	7050 3600 7350 3600
-Wire Wire Line
-	7350 3600 7350 3750
-Wire Wire Line
-	7050 3500 7400 3500
-Wire Wire Line
-	7400 3500 7400 3350
-Wire Wire Line
 	9750 1600 10250 1600
 Wire Wire Line
@@
 Wire Wire Line
 	3600 2000 7150 2000
-Connection ~ 7150 2550
 Wire Wire Line
 	3600 2100 6700 2100
 Wire Wire Line
 	6700 2100 6700 4400
-Connection ~ 7150 4400
 Wire Wire Line
 	4150 2800 4050 2800
@@
 We want to make source current from TINY to be <= 10 mA.\nSo we use MOC3043/MOC3063 - see last '3' here \nstands for modification with trigger current of 5 mA.\nThe Red LED is set up to drain less than 2 mA.
 $Comp
-L Screw_Terminal_01x02 J3
+L Screw_Terminal_01x02 J1
 U 1 1 5E7855C3
 P 10450 1500
-F 0 "J3" H 10450 1600 50  0000 C CNN
+F 0 "J1" H 10450 1600 50  0000 C CNN
 F 1 "Screw_Terminal_01x02" H 10450 1300 50  0000 C CNN
 F 2 "Connectors_Terminal_Blocks:TerminalBlock_Pheonix_MKDS1.5-2pol" H 10450 1500 50  0001 C CNN
@@
 	10250 1500 10150 1500
 $Comp
-L Screw_Terminal_01x02 J1
+L Screw_Terminal_01x02 J2
 U 1 1 5E786F25
 P 10650 3750
-F 0 "J1" H 10650 3850 50  0000 C CNN
+F 0 "J2" H 10650 3850 50  0000 C CNN
 F 1 "Screw_Terminal_01x02" H 10650 3550 50  0000 C CNN
 F 2 "Connectors_Terminal_Blocks:TerminalBlock_Pheonix_MKDS1.5-2pol" H 10650 3750 50  0001 C CNN
@@
 	1    0    0    1
 $EndComp
+$Comp
+L GND #PWR013
+U 1 1 5A12EDB6
+P 8300 3750
+F 0 "#PWR013" H 8300 3500 50  0001 C CNN
+F 1 "GND" H 8300 3600 50  0000 C CNN
+F 2 "" H 8300 3750 50  0001 C CNN
+F 3 "" H 8300 3750 50  0001 C CNN
+	1    8300 3750
+	1    0    0    -1
+$EndComp
+Wire Wire Line
+	7150 2000 7150 2550
 $EndSCHEMATC
